Commit message: Made bumblebee2 collision mesh a rectangle.

File: pointgrey_camera_description/urdf/pointgrey_bumblebee2.urdf.xacro (robot description, xacro)
@@ -69,7 +69,7 @@
       </visual>
       <collision>
-        <origin xyz="0 0 0" rpy="-1.5707 0 -1.5707"/>
+        <origin xyz="0 0 0" rpy="0 0 0"/>
         <geometry>
-          <mesh filename="package://pointgrey_camera_description/meshes/pointgrey_bumblebee2.dae"/>
+          <box size="0.04740 0.157 0.036"/>
         </geometry>
       </collision>
